File: flowerpower/flowerpower.kicad_pcb (KiCad board)
At the start: 2 copper layers, 16 parts

Commit message: Andringar
Routing:
- net N-000009: track 0.00 -> 63.0 mm
- net (no net): track 63.0 -> 0.00 mm
Other:
- board outline added: 42 x 84 mm
Changed lines of the file:
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@@
   (general
     (links 22)
-    (no_connects 15)
+    (no_connects 6)
     (area 27.965561 20.51055 45.127001 92.48945)
     (thickness 1.6)
-    (drawings 0)
+    (drawings 4)
     (tracks 24)
     (zones 0)
@@
     (pad_to_mask_clearance 0)
     (aux_axis_origin 0 0)
-    (visible_elements FFFFFFBF)
+    (visible_elements 7FFFFFFF)
     (pcbplotparams
       (layerselection 3178497)
@@
     (fp_arc (start 0.254 0) (end -1.905 0) (angle 90) (layer F.SilkS) (width 0.1524))
     (fp_arc (start 0.254 0) (end 2.413 0) (angle 90) (layer F.SilkS) (width 0.1524))
-    (pad 1 thru_hole circle (at -1.27 0) (size 1.6764 1.6764) (drill 0.8128)
+    (pad 1 thru_hole circle (at -1.27 0) (size 1.6764 1.6764) (drill 0.812799)
       (layers *.Cu *.Mask F.SilkS)
       (net 8 N-000007)
     )
-    (pad 2 thru_hole circle (at 1.27 0) (size 1.6764 1.6764) (drill 0.8128)
+    (pad 2 thru_hole circle (at 1.27 0) (size 1.6764 1.6764) (drill 0.812799)
       (layers *.Cu *.Mask F.SilkS)
       (net 2 N-0000010)
@@
     (fp_arc (start 0.254 0) (end -1.905 0) (angle 90) (layer F.SilkS) (width 0.1524))
     (fp_arc (start 0.254 0) (end 2.413 0) (angle 90) (layer F.SilkS) (width 0.1524))
-    (pad 1 thru_hole circle (at -1.27 0) (size 1.6764 1.6764) (drill 0.8128)
+    (pad 1 thru_hole circle (at -1.27 0) (size 1.6764 1.6764) (drill 0.812799)
       (layers *.Cu *.Mask F.SilkS)
       (net 9 N-000008)
     )
-    (pad 2 thru_hole circle (at 1.27 0) (size 1.6764 1.6764) (drill 0.8128)
+    (pad 2 thru_hole circle (at 1.27 0) (size 1.6764 1.6764) (drill 0.812799)
       (layers *.Cu *.Mask F.SilkS)
       (net 2 N-0000010)
@@
     (fp_arc (start 0.254 0) (end -1.905 0) (angle 90) (layer F.SilkS) (width 0.1524))
     (fp_arc (start 0.254 0) (end 2.413 0) (angle 90) (layer F.SilkS) (width 0.1524))
-    (pad 1 thru_hole circle (at -1.27 0) (size 1.6764 1.6764) (drill 0.8128)
+    (pad 1 thru_hole circle (at -1.27 0) (size 1.6764 1.6764) (drill 0.812799)
       (layers *.Cu *.Mask F.SilkS)
       (net 5 N-0000015)
     )
-    (pad 2 thru_hole circle (at 1.27 0) (size 1.6764 1.6764) (drill 0.8128)
+    (pad 2 thru_hole circle (at 1.27 0) (size 1.6764 1.6764) (drill 0.812799)
       (layers *.Cu *.Mask F.SilkS)
       (net 2 N-0000010)
@@
     (fp_arc (start 0.254 0) (end -1.905 0) (angle 90) (layer F.SilkS) (width 0.1524))
     (fp_arc (start 0.254 0) (end 2.413 0) (angle 90) (layer F.SilkS) (width 0.1524))
-    (pad 1 thru_hole circle (at -1.27 0) (size 1.6764 1.6764) (drill 0.8128)
+    (pad 1 thru_hole circle (at -1.27 0) (size 1.6764 1.6764) (drill 0.812799)
       (layers *.Cu *.Mask F.SilkS)
       (net 4 N-0000014)
     )
-    (pad 2 thru_hole circle (at 1.27 0) (size 1.6764 1.6764) (drill 0.8128)
+    (pad 2 thru_hole circle (at 1.27 0) (size 1.6764 1.6764) (drill 0.812799)
       (layers *.Cu *.Mask F.SilkS)
       (net 2 N-0000010)
@@
     (fp_arc (start 0.254 0) (end -1.905 0) (angle 90) (layer F.SilkS) (width 0.1524))
     (fp_arc (start 0.254 0) (end 2.413 0) (angle 90) (layer F.SilkS) (width 0.1524))
-    (pad 1 thru_hole circle (at -1.27 0) (size 1.6764 1.6764) (drill 0.8128)
+    (pad 1 thru_hole circle (at -1.27 0) (size 1.6764 1.6764) (drill 0.812799)
       (layers *.Cu *.Mask F.SilkS)
       (net 3 N-0000011)
     )
-    (pad 2 thru_hole circle (at 1.27 0) (size 1.6764 1.6764) (drill 0.8128)
+    (pad 2 thru_hole circle (at 1.27 0) (size 1.6764 1.6764) (drill 0.812799)
       (layers *.Cu *.Mask F.SilkS)
       (net 2 N-0000010)
@@
     (fp_arc (start 0.254 0) (end -1.905 0) (angle 90) (layer F.SilkS) (width 0.1524))
     (fp_arc (start 0.254 0) (end 2.413 0) (angle 90) (layer F.SilkS) (width 0.1524))
-    (pad 1 thru_hole circle (at -1.27 0) (size 1.6764 1.6764) (drill 0.8128)
+    (pad 1 thru_hole circle (at -1.27 0) (size 1.6764 1.6764) (drill 0.812799)
       (layers *.Cu *.Mask F.SilkS)
       (net 7 N-000003)
     )
-    (pad 2 thru_hole circle (at 1.27 0) (size 1.6764 1.6764) (drill 0.8128)
+    (pad 2 thru_hole circle (at 1.27 0) (size 1.6764 1.6764) (drill 0.812799)
       (layers *.Cu *.Mask F.SilkS)
       (net 2 N-0000010)
@@
     (fp_arc (start 0.254 0) (end -1.905 0) (angle 90) (layer F.SilkS) (width 0.1524))
     (fp_arc (start 0.254 0) (end 2.413 0) (angle 90) (layer F.SilkS) (width 0.1524))
-    (pad 1 thru_hole circle (at -1.27 0) (size 1.6764 1.6764) (drill 0.8128)
+    (pad 1 thru_hole circle (at -1.27 0) (size 1.6764 1.6764) (drill 0.812799)
       (layers *.Cu *.Mask F.SilkS)
       (net 1 N-000001)
     )
-    (pad 2 thru_hole circle (at 1.27 0) (size 1.6764 1.6764) (drill 0.8128)
+    (pad 2 thru_hole circle (at 1.27 0) (size 1.6764 1.6764) (drill 0.812799)
       (layers *.Cu *.Mask F.SilkS)
       (net 2 N-0000010)
@@
     (fp_arc (start 0.254 0) (end -1.905 0) (angle 90) (layer F.SilkS) (width 0.1524))
     (fp_arc (start 0.254 0) (end 2.413 0) (angle 90) (layer F.SilkS) (width 0.1524))
-    (pad 1 thru_hole circle (at -1.27 0) (size 1.6764 1.6764) (drill 0.8128)
+    (pad 1 thru_hole circle (at -1.27 0) (size 1.6764 1.6764) (drill 0.812799)
       (layers *.Cu *.Mask F.SilkS)
       (net 6 N-000002)
     )
-    (pad 2 thru_hole circle (at 1.27 0) (size 1.6764 1.6764) (drill 0.8128)
-      (layers *.Cu *.Mask F.SilkS)
-      (net 2 N-0000010)
-    )
-    (model discret/leds/led5_vertical_verde.wrl
-      (at (xyz 0 0 0))
-      (scale (xyz 1 1 1))
-      (rotate (xyz 0 0 0))
-    )
-  )
-  (segment (start 29 25) (end 29 88) (width 0.254) (layer B.Cu) (net 0))
-  (segment (start 36.73 70) (end 31 70) (width 0.254) (layer B.Cu) (net 1) (status 400000))
-  (segment (start 39.27 43) (end 45 43) (width 0.254) (layer B.Cu) (net 2) (status 400000))
-  (segment (start 39.27 52) (end 45 52) (width 0.254) (layer B.Cu) (net 2) (status 400000))
-  (segment (start 39.27 61) (end 45 61) (width 0.254) (layer B.Cu) (net 2) (status 400000))
-  (segment (start 39.27 70) (end 45 70) (width 0.254) (layer B.Cu) (net 2) (status 400000))
-  (segment (start 39.27 79) (end 45 79) (width 0.254) (layer B.Cu) (net 2) (status 400000))
+    (pad 2 thru_hole circle (at 1.27 0) (size 1.6764 1.6764) (drill 0.812799)
+      (layers *.Cu *.Mask F.SilkS)
+      (net 2 N-0000010)
+    )
+    (model discret/leds/led5_vertical_verde.wrl
+      (at (xyz 0 0 0))
+      (scale (xyz 1 1 1))
+      (rotate (xyz 0 0 0))
+    )
+  )
+  (gr_line (start 18 100) (end 18 16) (angle 90) (layer Edge.Cuts) (width 0.15))
+  (gr_line (start 60 100) (end 18 100) (angle 90) (layer Edge.Cuts) (width 0.15))
+  (gr_line (start 60 16) (end 60 100) (angle 90) (layer Edge.Cuts) (width 0.15))
+  (gr_line (start 18 16) (end 60 16) (angle 90) (layer Edge.Cuts) (width 0.15))
+  (segment (start 36.73 70) (end 31 70) (width 0.254) (layer B.Cu) (net 1))
+  (segment (start 39.27 43) (end 45 43) (width 0.254) (layer B.Cu) (net 2))
+  (segment (start 39.27 52) (end 45 52) (width 0.254) (layer B.Cu) (net 2))
+  (segment (start 39.27 61) (end 45 61) (width 0.254) (layer B.Cu) (net 2))
+  (segment (start 39.27 70) (end 45 70) (width 0.254) (layer B.Cu) (net 2))
+  (segment (start 39.27 79) (end 45 79) (width 0.254) (layer B.Cu) (net 2))
   (segment (start 45 34) (end 45 43) (width 0.254) (layer B.Cu) (net 2))
   (segment (start 45 43) (end 45 52) (width 0.254) (layer B.Cu) (net 2))
@@
   (segment (start 45 70) (end 45 79) (width 0.254) (layer B.Cu) (net 2))
   (segment (start 45 79) (end 45 88) (width 0.254) (layer B.Cu) (net 2))
-  (segment (start 45 88) (end 39.27 88) (width 0.254) (layer B.Cu) (net 2) (status 800000))
+  (segment (start 45 88) (end 39.27 88) (width 0.254) (layer B.Cu) (net 2))
   (segment (start 45 25) (end 45 34) (width 0.254) (layer B.Cu) (net 2))
-  (segment (start 39.27 25) (end 45 25) (width 0.254) (layer B.Cu) (net 2) (status 400000))
-  (segment (start 45 34) (end 39.27 34) (width 0.254) (layer B.Cu) (net 2) (status 800000))
-  (segment (start 36.73 88) (end 31 88) (width 0.254) (layer B.Cu) (net 3) (status 400000))
-  (segment (start 36.73 25) (end 31 25) (width 0.254) (layer B.Cu) (net 4) (status 400000))
-  (segment (start 36.73 34) (end 31 34) (width 0.254) (layer B.Cu) (net 5) (status 400000))
-  (segment (start 36.73 61) (end 31 61) (width 0.254) (layer B.Cu) (net 6) (status 400000))
-  (segment (start 36.73 79) (end 31 79) (width 0.254) (layer B.Cu) (net 7) (status 400000))
-  (segment (start 36.73 52) (end 31 52) (width 0.254) (layer B.Cu) (net 8) (status 400000))
-  (segment (start 36.73 43) (end 31 43) (width 0.254) (layer B.Cu) (net 9) (status 400000))
+  (segment (start 39.27 25) (end 45 25) (width 0.254) (layer B.Cu) (net 2))
+  (segment (start 45 34) (end 39.27 34) (width 0.254) (layer B.Cu) (net 2))
+  (segment (start 36.73 88) (end 31 88) (width 0.254) (layer B.Cu) (net 3))
+  (segment (start 36.73 25) (end 31 25) (width 0.254) (layer B.Cu) (net 4))
+  (segment (start 36.73 34) (end 31 34) (width 0.254) (layer B.Cu) (net 5))
+  (segment (start 36.73 61) (end 31 61) (width 0.254) (layer B.Cu) (net 6))
+  (segment (start 36.73 79) (end 31 79) (width 0.254) (layer B.Cu) (net 7))
+  (segment (start 36.73 52) (end 31 52) (width 0.254) (layer B.Cu) (net 8))
+  (segment (start 36.73 43) (end 31 43) (width 0.254) (layer B.Cu) (net 9))
+  (segment (start 29 25) (end 29 88) (width 0.254) (layer B.Cu) (net 10))
 )
